File: riffle-proto-0.1.brd (EAGLE design)
At the start: 62.2 x 18 mm, 15 parts

Commit message: update
Connections:
- net N$46: now also JP10.11
Changed lines of the file:
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@@
 </autorouter>
 <elements>
-<element name="JP6" library="microbuilder" package="1X11_ROUND_76" value="" x="22.86" y="4.572"/>
-<element name="JP7" library="microbuilder" package="1X11_ROUND_76" value="" x="22.86" y="2.032"/>
-<element name="JP3" library="microbuilder" package="1X11_ROUND_76" value="" x="22.86" y="12.192"/>
-<element name="JP5" library="microbuilder" package="1X11_ROUND_76" value="" x="22.86" y="7.112"/>
-<element name="JP4" library="microbuilder" package="1X11_ROUND_76" value="" x="22.86" y="9.652"/>
-<element name="JP1" library="microbuilder" package="1X11_ROUND_76" value="" x="22.86" y="17.272"/>
-<element name="JP2" library="microbuilder" package="1X11_ROUND_76" value="" x="22.86" y="14.732"/>
-<element name="SV2" library="con-lstb" package="MA07-2" value="" x="5.842" y="9.652" rot="R90">
+<element name="JP6" library="microbuilder" package="1X11_ROUND_76" value="" x="22.86" y="4.572" smashed="yes">
+<attribute name="VALUE" x="8.89" y="1.397" size="1.27" layer="27"/>
+</element>
+<element name="JP7" library="microbuilder" package="1X11_ROUND_76" value="" x="22.86" y="2.032" smashed="yes">
+<attribute name="VALUE" x="8.89" y="-1.143" size="1.27" layer="27"/>
+</element>
+<element name="JP3" library="microbuilder" package="1X11_ROUND_76" value="" x="22.86" y="12.192" smashed="yes">
+<attribute name="VALUE" x="8.89" y="9.017" size="1.27" layer="27"/>
+</element>
+<element name="JP5" library="microbuilder" package="1X11_ROUND_76" value="" x="22.86" y="7.112" smashed="yes">
+<attribute name="VALUE" x="8.89" y="3.937" size="1.27" layer="27"/>
+</element>
+<element name="JP4" library="microbuilder" package="1X11_ROUND_76" value="" x="22.86" y="9.652" smashed="yes">
+<attribute name="VALUE" x="8.89" y="6.477" size="1.27" layer="27"/>
+</element>
+<element name="JP1" library="microbuilder" package="1X11_ROUND_76" value="" x="22.86" y="17.272" smashed="yes">
+<attribute name="VALUE" x="8.89" y="14.097" size="1.27" layer="27"/>
+</element>
+<element name="JP2" library="microbuilder" package="1X11_ROUND_76" value="" x="22.86" y="14.732" smashed="yes">
+<attribute name="VALUE" x="8.89" y="11.557" size="1.27" layer="27"/>
+</element>
+<element name="SV2" library="con-lstb" package="MA07-2" value="" x="5.842" y="9.652" smashed="yes" rot="R90">
 <attribute name="MPN" value="" x="5.842" y="9.652" size="1.778" layer="27" rot="R90" display="off"/>
 <attribute name="MF" value="" x="5.842" y="9.652" size="1.778" layer="27" rot="R90" display="off"/>
 <attribute name="OC_FARNELL" value="unknown" x="5.842" y="9.652" size="1.778" layer="27" rot="R90" display="off"/>
 <attribute name="OC_NEWARK" value="unknown" x="5.842" y="9.652" size="1.778" layer="27" rot="R90" display="off"/>
-</element>
-<element name="JP8" library="microbuilder" package="1X11_ROUND_76" value="" x="51.054" y="17.272"/>
-<element name="JP9" library="microbuilder" package="1X11_ROUND_76" value="" x="51.054" y="14.732"/>
-<element name="JP10" library="microbuilder" package="1X11_ROUND_76" value="" x="51.054" y="12.192"/>
-<element name="JP11" library="microbuilder" package="1X11_ROUND_76" value="" x="51.054" y="9.652"/>
-<element name="JP12" library="microbuilder" package="1X11_ROUND_76" value="" x="51.054" y="7.112"/>
-<element name="JP13" library="microbuilder" package="1X11_ROUND_76" value="" x="51.054" y="4.572"/>
-<element name="JP14" library="microbuilder" package="1X11_ROUND_76" value="" x="51.054" y="2.032"/>
+<attribute name="VALUE" x="10.033" y="7.112" size="1.27" layer="27" ratio="10" rot="R90"/>
+</element>
+<element name="JP8" library="microbuilder" package="1X11_ROUND_76" value="" x="51.054" y="17.272" smashed="yes">
+<attribute name="VALUE" x="37.084" y="14.097" size="1.27" layer="27"/>
+</element>
+<element name="JP9" library="microbuilder" package="1X11_ROUND_76" value="" x="51.054" y="14.732" smashed="yes">
+<attribute name="VALUE" x="37.084" y="11.557" size="1.27" layer="27"/>
+</element>
+<element name="JP10" library="microbuilder" package="1X11_ROUND_76" value="" x="51.054" y="12.192" smashed="yes">
+<attribute name="VALUE" x="37.084" y="9.017" size="1.27" layer="27"/>
+</element>
+<element name="JP11" library="microbuilder" package="1X11_ROUND_76" value="" x="51.054" y="9.652" smashed="yes">
+<attribute name="VALUE" x="37.084" y="6.477" size="1.27" layer="27"/>
+</element>
+<element name="JP12" library="microbuilder" package="1X11_ROUND_76" value="" x="51.054" y="7.112" smashed="yes">
+<attribute name="VALUE" x="37.084" y="3.937" size="1.27" layer="27"/>
+</element>
+<element name="JP13" library="microbuilder" package="1X11_ROUND_76" value="" x="51.054" y="4.572" smashed="yes">
+<attribute name="VALUE" x="37.084" y="1.397" size="1.27" layer="27"/>
+</element>
+<element name="JP14" library="microbuilder" package="1X11_ROUND_76" value="" x="51.054" y="2.032" smashed="yes">
+<attribute name="VALUE" x="37.084" y="-1.143" size="1.27" layer="27"/>
+</element>
 </elements>
 <signals>
@@
 <wire x1="63.7794" y1="7.0866" x2="63.754" y2="7.112" width="0.254" layer="1"/>
 <wire x1="63.754" y1="14.732" x2="63.754" y2="9.652" width="0.254" layer="1"/>
+<contactref element="JP10" pad="11"/>
+<wire x1="63.754" y1="14.732" x2="63.754" y2="12.192" width="0" layer="19" extent="1-1"/>
 </signal>
 <signal name="N$24">
