File: riffle-proto-grove-1.3.sch (EAGLE design)
At the start: 22 parts, among them J10 A1, J9 A0

Commit message: update
Parts:
- removed J10: A1, Connector:TWIG-4P-2.0'90D'
- removed JP13, JP22, JP23, JP24, JP25, JP26, JP27, JP28: (no value), microbuilder:HEADER-1X670MIL
- added JP1, JP2, JP3, JP4, JP5: (no value), microbuilder:HEADER-1X770MIL
- added JP6, JP7: (no value), microbuilder:HEADER-1X2ROUND
Connections:
- new net N$12: JP15.1, JP15.2, JP15.3, JP15.4, JP15.5, JP15.6, JP15.7
- new net N$13: JP16.1, JP16.2, JP16.3, JP16.4, JP16.5, JP16.6, JP16.7
- new net N$14: JP17.1, JP17.2, JP17.3, JP17.4, JP17.5, JP17.6, JP17.7
- new net N$15: JP18.1, JP18.2, JP18.3, JP18.4, JP18.5, JP18.6, JP18.7
- new net N$16: JP19.1, JP19.2, JP19.3, JP19.4, JP19.5, JP19.6, JP19.7
- new net N$17: JP20.1, JP20.2, JP20.3, JP20.4, JP20.5, JP20.6, JP20.7
- new net N$18: JP21.1, JP21.2, JP21.3, JP21.4, JP21.5, JP21.6, JP21.7
- new net N$19: JP1.1, JP1.2, JP1.3, JP1.4, JP1.5, JP1.6, JP1.7
- new net N$20: JP2.1, JP2.2, JP2.3, JP2.4, JP2.5, JP2.6, JP2.7
- new net N$21: JP3.1, JP3.2, JP3.3, JP3.4, JP3.5, JP3.6, JP3.7
- new net N$22: JP4.1, JP4.2, JP4.3, JP4.4, JP4.5, JP4.6, JP4.7
- new net N$23: JP5.1, JP5.2, JP5.3, JP5.4, JP5.5, JP5.6, JP5.7
- new net N$24: JP6.1, JP6.2
- new net N$25: JP7.1, JP7.2
- new net N$8: JP10.1, JP10.2, JP10.3, JP10.4, JP10.5, JP10.6, JP10.7
- new net N$9: JP14.1, JP14.2, JP14.3, JP14.4, JP14.5, JP14.6, JP14.7
- net GND: no longer J10.4, J9.4
- net SCL: no longer J10.1, J9.1
- net SDA: no longer J10.2, J9.2
- net VCC: no longer J10.3, J9.3
Other:
- moved on the sheet: J9
